Commit message: URDF modified to add the gripper

File: ROS1/src/phantomx_pincher_arm/phantomx_pincher_arm_description/urdf/pincher_arm.urdf (robot description, URDF)
Before this commit: robot phantomx_pincher_arm, 7 links, 6 joints
Links:
- removed link gripper_link
- added link gripper_active2_link; collision mesh filename=package://phantomx_pincher_arm_description/meshes/PincherFi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; visual mesh filename=package://phantomx_pincher_arm_description/meshes/PincherFi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
- added link gripper_active_link; collision mesh filename=package://phantomx_pincher_arm_description/meshes/PincherFi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; visual mesh filename=package://phantomx_pincher_arm_description/meshes/PincherFi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
Joints:
- added joint gripper2_joint: type prismatic, parent arm_wrist_flex_link, child gripper_active2_link, origin xyz=0.070 0 0 rpy=0 0 0, axis 0 1 0, limit lower=-0.032 upper=-0.002 effort=30 velocity=0.5, mimic joint=gripper_link_joint multiplier=-1.0 offset=0.0
- joint gripper_link_joint: axis 1 0 0 -> 0 1 0; child gripper_link -> gripper_active_link; limit lower=-3.14 upper=3.14 effort=6 velocity=1 -> lower=0.002 upper=0.032 effort=30 velocity=0.5; origin xyz=0.110 0 0 rpy=0 0 0 -> xyz=0.070 0 0 rpy=0 0 0; type revolute -> prismatic
