Commit message: ROS2 bridge et ros2_control config added for a MockHardware

File: ROS2/src/phantomx_pincher_arm/phantomx_pincher_description/urdf/phantomx_pincher.urdf.xacro (robot description, xacro)
@@ -159,3 +159,31 @@
     </collision>
   </link>
+  <!-- ========================= -->
+  <!-- ROS 2 Control             -->
+  <!-- ========================= -->
+  <ros2_control name="PhantomXPincherSystem" type="system">
+    <hardware>
+      <plugin>mock_components/GenericSystem</plugin>
+    </hardware>
+    <joint name="arm_shoulder_pan_joint">
+      <command_interface name="position"/>
+      <state_interface name="position"/>
+    </joint>
+    <joint name="arm_bicep_joint">
+      <command_interface name="position"/>
+      <state_interface name="position"/>
+    </joint>
+    <joint name="arm_forearm_joint">
+      <command_interface name="position"/>
+      <state_interface name="position"/>
+    </joint>
+    <joint name="arm_wrist_flex_joint">
+      <command_interface name="position"/>
+      <state_interface name="position"/>
+    </joint>
+    <joint name="gripper_link_joint">
+      <command_interface name="position"/>
+      <state_interface name="position"/>
+    </joint>
+  </ros2_control>
 </robot>
